File: controller.sch (KiCad schematic (older format))
At the start: 64 parts, among them CON1 SD_Card, P1 ISP, P10 RS485, P2 BUTTONS, P3 OPEN_DRAIN, P4 POWER, P5 I2C1, P6 I2C2, P7 CONN_01X05, P8 THERMOCOUPLE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

Commit message: Put netlist and fottprint assignments into order, but something went hugely wrong -- 3V3 net replaces VCC net. FML
Parts:
- D2, D3, D4: footprint SMD_Packages:SOT-323 -> Housings_SOT-23_SOT-143_TSOT-6:SOT-23
- IC1: renamed from IC?; footprint TQFP32 -> Housings_QFP:TQFP-32_7x7mm_Pitch0.8mm
- RLY1: footprint (none) -> w_relay:relay_40.61
Connections:
- net at C20.2, C22.1, R12.2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: now also D4.1; no longer D4.2
- net at C20.1, C21.1, R7.2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: now also D4.2; no longer D4.1
Changed lines of the file:
@@
 P 10900 1300
 F 0 "R7" V 10980 1300 50  0000 C CNN
-F 1 "R" V 10907 1301 50  0000 C CNN
+F 1 "R" V 10900 1300 50  0000 C CNN
 F 2 "Resistors_SMD:R_0603_HandSoldering" V 10830 1300 30  0001 C CNN
 F 3 "" H 10900 1300 30  0000 C CNN
@@
 F 0 "RLY1" H 6200 5900 60  0000 C CNN
 F 1 "RELAY_40.61" H 6200 5300 60  0000 C CNN
-F 2 "" H 6200 5550 60  0001 C CNN
+F 2 "w_relay:relay_40.61" H 6200 5550 60  0001 C CNN
 F 3 "" H 6200 5550 60  0000 C CNN
 	1    6200 5650
@@
 L TVS-DUAL D4
 U 1 1 54F41A84
-P 11050 1500
-F 0 "D4" H 11050 1650 50  0000 C CNN
-F 1 "TVS-DUAL" H 11050 1150 50  0000 C CNN
-F 2 "SMD_Packages:SOT-323" H 11050 1500 60  0001 C CNN
-F 3 "" H 11050 1500 60  0000 C CNN
-	1    11050 1500
-	1    0    0    -1
+P 11050 1650
+F 0 "D4" H 11050 1800 50  0000 C CNN
+F 1 "TVS-DUAL" H 11100 1750 50  0000 C CNN
+F 2 "Housings_SOT-23_SOT-143_TSOT-6:SOT-23" H 11050 1650 60  0001 C CNN
+F 3 "" H 11050 1650 60  0000 C CNN
+	1    11050 1650
+	1    0    0    1
 $EndComp
 $Comp
 L GND #PWR053
 U 1 1 54F42988
-P 11400 1600
-F 0 "#PWR053" H 11400 1350 60  0001 C CNN
-F 1 "GND" H 11400 1450 60  0000 C CNN
-F 2 "" H 11400 1600 60  0000 C CNN
-F 3 "" H 11400 1600 60  0000 C CNN
-	1    11400 1600
+P 11400 1550
+F 0 "#PWR053" H 11400 1300 60  0001 C CNN
+F 1 "GND" H 11400 1400 60  0000 C CNN
+F 2 "" H 11400 1550 60  0000 C CNN
+F 3 "" H 11400 1550 60  0000 C CNN
+	1    11400 1550
 	1    0    0    -1
 $EndComp
@@
 F 0 "D3" H 10800 6400 50  0000 C CNN
 F 1 "TVS-DUAL" H 10800 5900 50  0000 C CNN
-F 2 "SMD_Packages:SOT-323" H 10800 6250 60  0001 C CNN
+F 2 "Housings_SOT-23_SOT-143_TSOT-6:SOT-23" H 10800 6250 60  0001 C CNN
 F 3 "" H 10800 6250 60  0000 C CNN
 	1    10800 6250
@@
 $EndComp
 Wire Wire Line
-	850  1100 1200 1100
-Wire Wire Line
-	1200 1100 1400 1100
-Wire Wire Line
-	1050 1300 1200 1300
-Wire Wire Line
-	1200 1300 1400 1300
-Wire Wire Line
-	650  1000 1200 1000
-Wire Wire Line
-	1200 1000 1400 1000
-Wire Wire Line
-	1200 800  1200 1000
-Wire Wire Line
-	1200 1000 1200 1100
-Wire Wire Line
-	1200 1100 1200 1300
+	850  1100 1400 1100
+Wire Wire Line
+	1050 1300 1400 1300
+Wire Wire Line
+	650  1000 1400 1000
+Wire Wire Line
+	1200 800  1200 1300
 Connection ~ 1200 1000
 Connection ~ 1200 1100
@@
 	1250 1600 1400 1600
 Wire Wire Line
-	650  1900 800  1900
-Wire Wire Line
-	800  1900 850  1900
-Wire Wire Line
-	850  1900 1050 1900
-Wire Wire Line
-	1050 1900 1250 1900
+	650  1900 1250 1900
 Wire Wire Line
 	1050 1600 1050 1900
@@
 	1200 3300 1400 3300
 Wire Wire Line
-	1200 3100 1200 3200
-Wire Wire Line
-	1200 3200 1200 3300
-Wire Wire Line
-	1200 3300 1200 3350
+	1200 3100 1200 3350
 Wire Wire Line
 	1400 3200 1200 3200
@@
 	3300 1700 4150 1700
 Wire Wire Line
-	4150 2000 4450 2000
-Wire Wire Line
-	4450 2000 4750 2000
+	4150 2000 4750 2000
 Wire Wire Line
 	4450 2000 4450 2000
@@
 	3300 2450 5050 2450
 Wire Wire Line
-	9950 1950 10150 1950
-Wire Wire Line
-	10150 1950 10400 1950
-Wire Wire Line
-	10400 1950 10750 1950
+	9950 1950 10750 1950
 Connection ~ 10150 1550
 Connection ~ 10150 1950
@@
 	9950 1550 10150 1550
 Wire Wire Line
-	10150 1300 10150 1550
-Wire Wire Line
-	10150 1550 10150 1600
-Wire Wire Line
-	10150 1300 10400 1300
-Wire Wire Line
-	10400 1300 10750 1300
+	10150 1300 10150 1600
+Wire Wire Line
+	10150 1300 10750 1300
 Connection ~ 10400 1950
 Connection ~ 10400 1300
 Wire Wire Line
-	650  4700 1100 4700
-Wire Wire Line
-	1100 4700 1500 4700
-Wire Wire Line
-	1500 4700 1900 4700
-Wire Wire Line
-	1900 4700 2200 4700
+	650  4700 2200 4700
 Wire Wire Line
 	1500 4600 1500 4700
 Connection ~ 1500 4700
 Wire Wire Line
-	2700 4600 3100 4600
-Wire Wire Line
-	3100 4600 3500 4600
+	2700 4600 3500 4600
 Wire Wire Line
 	3100 4600 3100 4600
@@
 Connection ~ 9450 650
 Wire Wire Line
-	2350 6550 2800 6550
-Wire Wire Line
-	2800 6550 3400 6550
-Wire Wire Line
-	3400 6550 4150 6550
-Wire Wire Line
-	4150 6550 4200 6550
-Wire Wire Line
-	3200 6650 3650 6650
-Wire Wire Line
-	3650 6650 4100 6650
-Wire Wire Line
-	4100 6650 4200 6650
-Wire Wire Line
-	3200 6750 3800 6750
-Wire Wire Line
-	3800 6750 4050 6750
-Wire Wire Line
-	4050 6750 4200 6750
-Wire Wire Line
-	3400 6850 4000 6850
-Wire Wire Line
-	4000 6850 4200 6850
-Wire Wire Line
-	4150 6250 4150 6550
-Wire Wire Line
-	4150 6550 4150 7200
+	2350 6550 4200 6550
+Wire Wire Line
+	3200 6650 4200 6650
+Wire Wire Line
+	3200 6750 4200 6750
+Wire Wire Line
+	3400 6850 4200 6850
+Wire Wire Line
+	4150 6250 4150 7200
 Wire Wire Line
 	4150 7200 4200 7200
@@
 	1600 7050 1250 7050
 Wire Wire Line
-	9850 5700 10450 5700
-Wire Wire Line
-	10450 5700 10900 5700
-Wire Wire Line
-	10900 5700 11500 5700
+	9850 5700 11500 5700
 Wire Wire Line
 	9850 5900 9850 6800
 Wire Wire Line
-	9850 6800 10600 6800
-Wire Wire Line
-	10600 6800 10800 6800
-Wire Wire Line
-	10800 6800 10950 6800
+	9850 6800 10950 6800
 Wire Wire Line
 	9450 4800 9600 4800
@@
 Connection ~ 3800 6750
 Wire Wire Line
-	3650 6100 3750 6100
-Wire Wire Line
-	3750 6100 3800 6100
+	3650 6100 3800 6100
 Wire Wire Line
 	3750 6000 3750 6100
@@
 	5700 6450 6000 6450
 Wire Wire Line
-	6000 6350 6000 6450
-Wire Wire Line
-	6000 6450 6000 6500
+	6000 6350 6000 6500
 Connection ~ 6000 6450
 Wire Wire Line
@@
 	6350 5950 7250 5950
 Wire Wire Line
-	7900 3750 8050 3750
-Wire Wire Line
-	8050 3750 8750 3750
+	7900 3750 8750 3750
 Wire Wire Line
 	8200 3650 8750 3650
@@
 	8650 4050 8750 4050
 Wire Wire Line
-	8200 3450 8350 3450
-Wire Wire Line
-	8350 3450 8750 3450
+	8200 3450 8750 3450
 Wire Wire Line
 	8750 3850 8300 3850
 Wire Wire Line
-	8200 3650 8200 3950
-Wire Wire Line
-	8200 3950 8200 4050
+	8200 3650 8200 4050
 Wire Wire Line
 	8750 3550 8200 3550
@@
 Connection ~ 6350 2650
 Wire Wire Line
-	8100 5250 8550 5250
-Wire Wire Line
-	8550 5250 8650 5250
+	8100 5250 8650 5250
 Wire Wire Line
 	8650 5250 8650 4050
@@
 	8250 4750 8250 5050
 Wire Wire Line
-	8250 2700 8700 2700
-Wire Wire Line
-	8700 2700 8800 2700
+	8250 2700 8800 2700
 Wire Wire Line
 	8800 2700 8800 1650
@@
 F 0 "D2" H 10600 7450 50  0000 C CNN
 F 1 "TVS-DUAL" H 10600 6950 50  0000 C CNN
-F 2 "SMD_Packages:SOT-323" H 10600 7300 60  0001 C CNN
+F 2 "Housings_SOT-23_SOT-143_TSOT-6:SOT-23" H 10600 7300 60  0001 C CNN
 F 3 "" H 10600 7300 60  0000 C CNN
 	1    10600 7300
@@
 Wire Wire Line
 	2800 6950 2800 6850
-Wire Wire Line
-	5700 6450 5700 6450
-$Comp
-L ATMEGA328P-A IC?
+$Comp
+L ATMEGA328P-A IC1
 U 1 1 5521429B
 P 2300 2100
-F 0 "IC?" H 1550 3350 40  0000 L BNN
+F 0 "IC1" H 1550 3350 40  0000 L BNN
 F 1 "ATMEGA328P-A" H 2700 700 40  0000 L BNN
-F 2 "TQFP32" H 2300 2100 30  0000 C CIN
+F 2 "Housings_QFP:TQFP-32_7x7mm_Pitch0.8mm" H 2300 2100 30  0000 C CIN
 F 3 "" H 2300 2100 60  0000 C CNN
 	1    2300 2100

Commit message: Fix netlist problem - update custom tuded ICs: U3 power connections are visible, U5 pin ordering more convenient. Saved cymbol changes to the local cache, not clear if this will help thoug..
Connections:
- net RXD: now also U5.1 (RO); no longer U5.4 (DI)
- net TXD: now also U5.4 (DI); no longer U5.1 (RO)
- net VCC renamed +12V

Commit message: Swap TVS pins again. Add pullup resistors to CS lines.
Parts:
- added R15, R16: 10k, Resistors_SMD:R_0603_HandSoldering, symbol R
Connections:
- net +5V: now also R15.1, R16.1
- net CS_SD: now also R16.2
- net CS_TC: now also R15.2
- net at C20.2, C22.1, R12.2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: now also D4.2; no longer D4.1
- net at C20.1, C21.1, R7.2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: now also D4.1; no longer D4.2
